File: Hardware/KiCad/GBR-4L/GBR-4L.kicad_sch (KiCad schematic)
At the start: 0 parts

Commit message: わかんないけど
Other:
- added sheet LED_RESET (LED_RESET.kicad_sch)
- added sheet LTE_SLOT1 (LTE_SLOT1.kicad_sch)
- added sheet LTE_SLOT2 (LTE_SLOT2.kicad_sch)
- added sheet LTE_SLOT3 (LTE_SLOT3.kicad_sch)
- added sheet LTE_SLOT4 (LTE_SLOT4.kicad_sch)
- added sheet Power (Power_sch.kicad_sch)
- added sheet SIM (SIM.kicad_sch)
- added sheet USB (USB.kicad_sch)
