File: Hardware/KiCad/GBR-4L/LED_RESET.kicad_sch (KiCad schematic)
At the start: 0 parts

Commit message: Add modem status and local controls
Parts:
- added D911: MODEM 1 STATUS GREEN, LED_SMD:LED_0603_1608Metric, symbol Device:LED
- added D921: MODEM 2 STATUS GREEN, LED_SMD:LED_0603_1608Metric, symbol Device:LED
- added D931: MODEM 3 STATUS GREEN, LED_SMD:LED_0603_1608Metric, symbol Device:LED
- added D941: MODEM 4 STATUS GREEN, LED_SMD:LED_0603_1608Metric, symbol Device:LED
- added Q911, Q921, Q931, Q941: MMBT3906, Package_TO_SOT_SMD:SOT-23, symbol Transistor_BJT:Q_PNP_BEC
- added R911, R912, R913, R921, R922, R923, R931, R932, R933, R941, R942, R943: 10k, Resistor_SMD:R_0603_1608Metric, symbol Device:R
- added R914, R924, R934, R944: 100k, Resistor_SMD:R_0603_1608Metric, symbol Device:R
- added R915, R925, R935, R945: 1k, Resistor_SMD:R_0603_1608Metric, symbol Device:R
- added SW911: MODEM 1 RESET, Button_Switch_SMD:SW_SPST_TL3305A, symbol Switch:SW_Push
- added SW912: MODEM 1 RF DISABLE, Button_Switch_SMD:SW_SPST_TL3305A, symbol Switch:SW_Push
- added SW921: MODEM 2 RESET, Button_Switch_SMD:SW_SPST_TL3305A, symbol Switch:SW_Push
- added SW922: MODEM 2 RF DISABLE, Button_Switch_SMD:SW_SPST_TL3305A, symbol Switch:SW_Push
- added SW931: MODEM 3 RESET, Button_Switch_SMD:SW_SPST_TL3305A, symbol Switch:SW_Push
- added SW932: MODEM 3 RF DISABLE, Button_Switch_SMD:SW_SPST_TL3305A, symbol Switch:SW_Push
- added SW941: MODEM 4 RESET, Button_Switch_SMD:SW_SPST_TL3305A, symbol Switch:SW_Push
- added SW942: MODEM 4 RF DISABLE, Button_Switch_SMD:SW_SPST_TL3305A, symbol Switch:SW_Push
Connections:
- new net +3V3_M1: Q911.2 (E), R911.1, R912.1, R914.1
- new net +3V3_M2: Q921.2 (E), R921.1, R922.1, R924.1
- new net +3V3_M3: Q931.2 (E), R931.1, R932.1, R934.1
- new net +3V3_M4: Q941.2 (E), R941.1, R942.1, R944.1
- new net GND: D911.1 (K), D921.1 (K), D931.1 (K), D941.1 (K), SW911.2, SW912.2, SW921.2, SW922.2, SW931.2, SW932.2, SW941.2, SW942.2
- new net M1_LED_ANODE: D911.2 (A), R915.2
- new net M1_LED_BASE: Q911.1 (B), R913.2, R914.2
- new net M1_LED_SOURCE: Q911.3 (C), R915.1
- new net M1_RESET_CTRL#: R911.2, SW911.1
- new net M1_WWAN_LED#: R913.1
- new net M1_W_DISABLE_CTRL#: R912.2, SW912.1
- new net M2_LED_ANODE: D921.2 (A), R925.2
- new net M2_LED_BASE: Q921.1 (B), R923.2, R924.2
- new net M2_LED_SOURCE: Q921.3 (C), R925.1
- new net M2_RESET_CTRL#: R921.2, SW921.1
- new net M2_WWAN_LED#: R923.1
- new net M2_W_DISABLE_CTRL#: R922.2, SW922.1
- new net M3_LED_ANODE: D931.2 (A), R935.2
- new net M3_LED_BASE: Q931.1 (B), R933.2, R934.2
- new net M3_LED_SOURCE: Q931.3 (C), R935.1
- new net M3_RESET_CTRL#: R931.2, SW931.1
- new net M3_WWAN_LED#: R933.1
- new net M3_W_DISABLE_CTRL#: R932.2, SW932.1
- new net M4_LED_ANODE: D941.2 (A), R945.2
- new net M4_LED_BASE: Q941.1 (B), R943.2, R944.2
- new net M4_LED_SOURCE: Q941.3 (C), R945.1
- new net M4_RESET_CTRL#: R941.2, SW941.1
- new net M4_WWAN_LED#: R943.1
- new net M4_W_DISABLE_CTRL#: R942.2, SW942.1
Other:
- note added: "Do not operate RESET or RF-disable controls while the corresponding modem rail is off."
- note added: "MODEM 1"
- note added: "MODEM 2"
- note added: "MODEM 3"
- note added: "MODEM 4"
- note added: "MODEM STATUS AND LOCAL CONTROLS"
- note added: "RESET# and W_DISABLE1# default high from the associated modem rail; buttons assert each signal low."
- note added: "Switch footprints are prototype defaults. Confirm actuator access and enclosure clearance before placement freeze."
- note added: "WWAN_LED# is buffered by a PNP high-side stage so the modem pin only sinks base current."
- title: (none) -> GBR-4L modem status and local controls

Commit message: Add connector footprints and initial PCB packing
Parts:
- SW911, SW912, SW921, SW922, SW931, SW932, SW941, SW942: footprint Button_Switch_SMD:SW_SPST_TL3305A -> Button_Switch_SMD:SW_SPST_B3U-1000P
