File: Hardware/KiCad/GBR-4L/Power_sch.kicad_sch (KiCad schematic)
At the start: 0 parts

Commit message: Add protected input and five 3.3 V rails
Parts:
- added C701: 220uF 25V, Capacitor_SMD:C_Elec_10x10.2, symbol Device:C
- added C702: 10uF 25V, Capacitor_SMD:C_1210_3225Metric, symbol Device:C
- added C703, C725, C745, C765, C785, C805: 100nF 50V, Capacitor_SMD:C_0603_1608Metric, symbol Device:C
- added C721, C741, C761, C781, C801: 100nF, Capacitor_SMD:C_0603_1608Metric, symbol Device:C
- added C722, C723, C742, C743, C762, C763, C782, C783, C802, C803: 22uF 16V X5R, Capacitor_SMD:C_0805_2012Metric, symbol Device:C
- added C724, C744, C764, C784, C804: 10uF 25V, Capacitor_SMD:C_0805_2012Metric, symbol Device:C
- added D701: SMBJ15A, Diode_SMD:D_SMB, symbol Device:D_TVS
- added D702: 12V, Diode_SMD:D_SOD-123, symbol Device:D_Zener
- added F701: 5A time-delay, Fuse:Fuseholder_Blade_ATO_Littelfuse_Pudenz_2_Pin, symbol Device:Fuse
- added J701: 12V INPUT 5A, TerminalBlock_Phoenix:TerminalBlock_Phoenix_MKDS-1,5-2_1x02_P5.00mm_Horizontal, symbol Connector_Generic:Conn_01x02
- added L721, L741, L761, L781, L801: 4.7uH Isat>=4A, Inductor_SMD:L_7.3x7.3_H3.5, symbol Device:L
- added Q701: 30V P-MOSFET low-RDS(on), Package_TO_SOT_SMD:TO-252-2, symbol Transistor_FET:Q_PMOS_GSD
- added R701: 100k, Resistor_SMD:R_0603_1608Metric, symbol Device:R
- added R721, R741, R761, R781, R801: 31.6k 1%, Resistor_SMD:R_0603_1608Metric, symbol Device:R
- added R722, R742, R762, R782, R802: 10.0k 1%, Resistor_SMD:R_0603_1608Metric, symbol Device:R
- added R723, R743, R763, R783: 174k 1%, Resistor_SMD:R_0603_1608Metric, symbol Device:R
- added R724, R744, R764, R784: 36.5k 1%, Resistor_SMD:R_0603_1608Metric, symbol Device:R
- added U721, U741, U761, U781, U801: TPS56339DDCR, Package_TO_SOT_SMD:SOT-23-6, symbol Regulator_Switching:TPS56339DDC
Connections:
- new net +12V_FUSED: D701.1 (A1), F701.2, Q701.3 (D)
- new net +12V_IN: F701.1, J701.1 (Pin_1)
- new net +12V_PROTECTED: C701.1, C702.1, C703.1, C724.1, C725.1, C744.1, C745.1, C764.1, C765.1, C784.1, C785.1, C804.1, C805.1, D702.1 (K), Q701.2 (S), R723.1, R743.1, R763.1, R783.1, U721.3 (VIN), U741.3 (VIN), U761.3 (VIN), U781.3 (VIN), U801.3 (VIN), U801.5 (EN)
- new net +3V3_M1: C722.1, C723.1, L721.2, R721.1
- new net +3V3_M2: C742.1, C743.1, L741.2, R741.1
- new net +3V3_M3: C762.1, C763.1, L761.2, R761.1
- new net +3V3_M4: C782.1, C783.1, L781.2, R781.1
- new net +3V3_SYS: C802.1, C803.1, L801.2, R801.1
- new net BOOT_1: C721.1, U721.6 (BOOT)
- new net BOOT_2: C741.1, U741.6 (BOOT)
- new net BOOT_3: C761.1, U761.6 (BOOT)
- new net BOOT_4: C781.1, U781.6 (BOOT)
- new net BOOT_5: C801.1, U801.6 (BOOT)
- new net FB_1: R721.2, R722.1, U721.4 (FB)
- new net FB_2: R741.2, R742.1, U741.4 (FB)
- new net FB_3: R761.2, R762.1, U761.4 (FB)
- new net FB_4: R781.2, R782.1, U781.4 (FB)
- new net FB_5: R801.2, R802.1, U801.4 (FB)
- new net GND: C701.2, C702.2, C703.2, C722.2, C723.2, C724.2, C725.2, C742.2, C743.2, C744.2, C745.2, C762.2, C763.2, C764.2, C765.2, C782.2, C783.2, C784.2, C785.2, C802.2, C803.2, C804.2, C805.2, D701.2 (A2), J701.2 (Pin_2), R701.2, R722.2, R724.2, R742.2, R744.2, R762.2, R764.2, R782.2, R784.2, R802.2, U721.1 (GND), U741.1 (GND), U761.1 (GND), U781.1 (GND), U801.1 (GND)
- new net M1_PWR_EN: R723.2, R724.1, U721.5 (EN)
- new net M2_PWR_EN: R743.2, R744.1, U741.5 (EN)
- new net M3_PWR_EN: R763.2, R764.1, U761.5 (EN)
- new net M4_PWR_EN: R783.2, R784.1, U781.5 (EN)
- new net SW_1: C721.2, L721.1, U721.2 (SW)
- new net SW_2: C741.2, L741.1, U741.2 (SW)
- new net SW_3: C761.2, L761.1, U761.2 (SW)
- new net SW_4: C781.2, L781.1, U781.2 (SW)
- new net SW_5: C801.2, L801.1, U801.2 (SW)
- new net VIN_PMOS_GATE: D702.2 (A), Q701.1 (G), R701.1
Other:
- note added: "12 V INPUT AND FIVE INDEPENDENT 3.3 V BUCK REGULATORS"
- note added: "BUCK 1: +3V3_M1"
- note added: "BUCK 2: +3V3_M2"
- note added: "BUCK 3: +3V3_M3"
- note added: "BUCK 4: +3V3_M4"
- note added: "BUCK 5: +3V3_SYS"
- note added: "Confirm the final MOSFET SOA, RDS(on), thermal rise and connector current rating before layout release."
- note added: "Each 3.3 V channel uses TI's recommended 31.6k/10k feedback divider, 4.7uH inductor and 2x22uF output network."
- note added: "Input protection: fuse, TVS and high-side P-MOS reverse-polarity stage."
- note added: "Modem EN nets default high via the UVLO divider and must be controlled only by open-drain/open-collector outputs."
- note added: "Prototype validation: stagger starts, measure 100mVpp maximum at every EM7565 socket, and test 2.5A inrush/load steps."
- note added: "TPS56339: 4.5–24 V input, 3 A output, 500 kHz, internal compensation and 5 ms soft-start."
- title: (none) -> GBR-4L power input and five 3.3 V rails

Commit message: Add connector footprints and initial PCB packing
Parts:
- removed U721, U741, U761, U781, U801: TPS56339DDCR, Package_TO_SOT_SMD:SOT-23-6, symbol Regulator_Switching:TPS56339DDC
- added U21, U22, U23, U24, U25: TPS56339DDCR, Package_TO_SOT_SMD:SOT-23-6, symbol Regulator_Switching:TPS56339DDC
Connections:
- net +12V_PROTECTED: now also U21.3 (VIN), U22.3 (VIN), U23.3 (VIN), U24.3 (VIN), U25.3 (VIN), U25.5 (EN)
- net BOOT_1: now also U21.6 (BOOT)
- net BOOT_2: now also U22.6 (BOOT)
- net BOOT_3: now also U23.6 (BOOT)
- net BOOT_4: now also U24.6 (BOOT)
- net BOOT_5: now also U25.6 (BOOT)
- net FB_1: now also U21.4 (FB)
- net FB_2: now also U22.4 (FB)
- net FB_3: now also U23.4 (FB)
- net FB_4: now also U24.4 (FB)
- net FB_5: now also U25.4 (FB)
- net GND: now also U21.1 (GND), U22.1 (GND), U23.1 (GND), U24.1 (GND), U25.1 (GND)
- net M1_PWR_EN: now also U21.5 (EN)
- net M2_PWR_EN: now also U22.5 (EN)
- net M3_PWR_EN: now also U23.5 (EN)
- net M4_PWR_EN: now also U24.5 (EN)
- net SW_1: now also U21.2 (SW)
- net SW_2: now also U22.2 (SW)
- net SW_3: now also U23.2 (SW)
- net SW_4: now also U24.2 (SW)
- net SW_5: now also U25.2 (SW)
